File: poormans73_hpf.sch (KiCad schematic (older format))
At the start: 39 parts, among them SW3 SW_DPDT_x2, SW4 SW_Rotary3x4, U4 NE5532, U5 NE5532

Commit message: completed HPF
added HPF measurements, updated schematics
Parts:
- renumbered C41 to C1, C34 to C10, C37 to C11, C27 to C12, C28 to C13, C29 to C14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
Connections:
- wire segments 114 -> 116
